Commit message: split sim and nav packages

File: asb_webots/resource/asb_webots_robot.urdf (robot description, URDF)
Before this commit: robot asb_webots_robot, 0 links, 0 joints
Links:
- added link base_footprint
- added link base_link; visual cylinder length=0.10 radius=0.20
- added link base_scan; visual cylinder length=0.05 radius=0.05
- added link gps_link
- added link wheel_left_link; visual cylinder length=0.05 radius=0.05
- added link wheel_right_link; visual cylinder length=0.05 radius=0.05
Joints:
- added joint base_joint: type fixed, parent base_footprint, child base_link, origin xyz=0 0 0.010 rpy=0 0 0
- added joint gps_joint: type fixed, parent base_link, child gps_link, origin xyz=0 0 0 rpy=0 0 0
- added joint scan_joint: type fixed, parent base_link, child base_scan, origin xyz=0 0 0.07 rpy=0 0 0
- added joint wheel_left_joint: type continuous, parent base_link, child wheel_left_link, origin xyz=0.0 0.144 0.023 rpy=-1.57 0 0, axis 0 0 1
- added joint wheel_right_joint: type continuous, parent base_link, child wheel_right_link, origin xyz=0.0 -0.144 0.023 rpy=-1.57 0 0, axis 0 0 1
