Commit message: added testing with dummy node and added current and temp conversion

File: asb_ros2_control/description/ros2_control/asb.ros2_control.xacro (robot description, xacro)
@@ -1,22 +1,25 @@
 <?xml version="1.0"?>
 <robot xmlns:xacro="http://www.ros.org/wiki/xacro">
-  <xacro:macro name="asb_ros2_control" params="name prefix">
+  <xacro:macro name="asb_ros2_control" params="name prefix test">
     <ros2_control name="${name}" type="system">
       <hardware>
         <plugin>asb_ros2_control/ASBSystemHardware</plugin>
         <param name="canopen_node_config">$(find asb_ros2_control)/config/GCU.dcf</param>
-        <param name="can_interface_name">vcan0</param>
+        <xacro:if value="${test}">
+          <param name="can_interface_name">vcan0</param>
+        </xacro:if>
+        <xacro:unless value="${test}">
+          <param name="can_interface_name">can0</param>
+        </xacro:unless>
         <param name="tracks_maximum_velocity_rpm">2400</param>
-        <!--        <param name="loop_rate">50</param>  TODO ? -->
-        <!--        <param name="timeout">50</param>  TODO ? -->
-        <param name="${prefix}left_track_joint_name">left_wheel_joint</param>
-        <param name="${prefix}right_track_joint_name">right_wheel_joint</param>
+        <param name="left_track_joint_name">left_wheel_joint</param>
+        <param name="right_track_joint_name">right_wheel_joint</param>
       </hardware>
-      <joint name="${prefix}left_wheel_joint">
+      <joint name="left_wheel_joint">
         <state_interface name="position"/>
         <state_interface name="velocity"/>
         <command_interface name="velocity"/>
       </joint>
-      <joint name="${prefix}right_wheel_joint">
+      <joint name="right_wheel_joint">
         <state_interface name="position"/>
         <state_interface name="velocity"/>

File: asb_ros2_control/description/urdf/asb_test.urdf.xacro (robot description, xacro)
@@ -9,4 +9,4 @@
   <xacro:include filename="$(find asb_ros2_control)/ros2_control/asb.ros2_control.xacro" />
 <!--  <xacro:diffbot prefix="$(arg prefix)" />-->
-  <xacro:asb_ros2_control name="asb" prefix="$(arg prefix)" test="false" />
+  <xacro:asb_ros2_control name="asb" prefix="$(arg prefix)" test="true" />
 </robot>

Commit message: added fan motor and pump command to HW interface

File: asb_ros2_control/description/ros2_control/asb.ros2_control.xacro (robot description, xacro)
@@ -29,4 +29,9 @@
         <command_interface name="velocity"/>
       </joint>
+      <joint name="fan_motor_joint"> <!-- in fan_motor_joint the velocity is in RPM and the position in revolutions -->
+        <state_interface name="position"/>
+        <state_interface name="velocity"/>
+        <command_interface name="velocity"/>
+      </joint>
       <gpio name="control_system_state">
         <state_interface name="vcu_comm_ok"/>
@@ -35,4 +40,6 @@
         <state_interface name="software_emergency_stop"/>
         <command_interface name="set_software_emergency_stop"/>
+        <state_interface name="pump_state"/>
+        <command_interface name="pump_command"/>
         <state_interface name="left_motor_controller_temperature"/>
         <state_interface name="left_motor_temperature"/>
@@ -41,5 +48,4 @@
         <state_interface name="right_motor_temperature"/>
         <state_interface name="right_motor_battery_current"/>
-        <state_interface name="fan_motor_rpm"/>
         <state_interface name="fan_motor_controller_temperature"/>
         <state_interface name="fan_motor_temperature"/>

Commit message: fixed fan max rpm and tracks joint names

File: asb_ros2_control/description/ros2_control/asb.ros2_control.xacro (robot description, xacro)
@@ -16,13 +16,12 @@
         </xacro:unless>
         <param name="tracks_maximum_velocity_rpm">2400</param>
-        <param name="left_track_joint_name">left_wheel_joint</param>
-        <param name="right_track_joint_name">right_wheel_joint</param>
+        <param name="fan_maximum_velocity_rpm">800</param>
       </hardware>
-      <joint name="left_wheel_joint">
+      <joint name="left_track_joint">
         <state_interface name="position"/>
         <state_interface name="velocity"/>
         <command_interface name="velocity"/>
       </joint>
-      <joint name="right_wheel_joint">
+      <joint name="right_track_joint">
         <state_interface name="position"/>
         <state_interface name="velocity"/>

Commit message: using webots for gnss navigation

File: asb_ros2_control/description/ros2_control/asb.ros2_control.xacro (robot description, xacro)
@@ -1,5 +1,5 @@
 <?xml version="1.0"?>
 <robot xmlns:xacro="http://www.ros.org/wiki/xacro">
-  <xacro:macro name="asb_ros2_control" params="name prefix test">
+  <xacro:macro name="asb_ros2_control" params="name test">
     <ros2_control name="${name}" type="system">
       <hardware>

File: asb_ros2_control/description/urdf/asb.materials.xacro (robot description, xacro)
@@ -29,3 +29,12 @@
     <color rgba="1.0 1.0 1.0 1.0"/>
   </material>
+  <material name="tire_color">
+      <color rgba="0.3 0.3 0.3 1.0"/>
+  </material>
+  <material name="base_color">
+      <color rgba="0.4 0.4 0.4 1.0"/>
+  </material>
+  <material name="lidar_color">
+      <color rgba="0.0 0.0 0.8 1.0"/>
+  </material>
 </robot>

File: asb_ros2_control/description/urdf/asb.urdf.xacro (robot description, xacro)
@@ -1,13 +1,11 @@
 <?xml version="1.0"?>
-<!-- Basic differential drive mobile base -->
 <robot xmlns:xacro="http://www.ros.org/wiki/xacro" name="asb_robot">
-  <xacro:arg name="prefix" default="" />
+<!--  <xacro:arg name="prefix" default="" />-->
   <xacro:arg name="test" default="false" />
   <xacro:include filename="$(find asb_ros2_control)/urdf/asb_description.urdf.xacro" />
-  <!-- Import Rviz colors -->
   <xacro:include filename="$(find asb_ros2_control)/urdf/asb.materials.xacro" />
-  <!-- Import asb ros2_control description -->
   <xacro:include filename="$(find asb_ros2_control)/ros2_control/asb.ros2_control.xacro" />
-  <xacro:asb prefix="$(arg prefix)" />
-  <xacro:asb_ros2_control name="asb" prefix="$(arg prefix)" test="$(arg test)" />
+  <xacro:asb_description />
+<!--  <xacro:asb prefix="$(arg prefix)" />-->
+  <xacro:asb_ros2_control name="asb" test="$(arg test)" />
 </robot>

File: asb_ros2_control/description/urdf/asb_description.urdf.xacro (robot description, xacro)
@@ -1,5 +1,6 @@
 <?xml version="1.0"?>
 <robot xmlns:xacro="http://www.ros.org/wiki/xacro">
-  <xacro:macro name="asb" params="prefix">
+  <xacro:macro name="asb_description">
+<!--  <xacro:macro name="asb" params="prefix">-->
     <!-- Constants for robot dimensions -->
     <xacro:property name="PI" value="3.1415926535897931"/>
@@ -13,5 +14,12 @@
     <xacro:property name="z_offset" value="-${base_height/2}" /> <!-- Space btw top of beam and each joint -->
     <!-- Base Link -->
-    <link name="${prefix}base_link">
+    <link name="base_footprint"/>
+    <joint name="base_joint" type="fixed">
+        <parent link="base_footprint"/>
+        <child link="base_link" />
+        <origin xyz="0 0 0.010" rpy="0 0 0"/>
+    </joint>
+    <!-- Base Link -->
+    <link name="base_link">
       <collision>
         <origin xyz="0 0 ${base_height/2}" rpy="0 0 0"/>
@@ -28,7 +36,7 @@
       </visual>
     </link>
-    <joint name="${prefix}left_wheel_joint" type="continuous">
-      <parent link="${prefix}base_link"/>
-      <child link="${prefix}left_wheel"/>
+    <joint name="left_wheel_joint" type="continuous">
+      <parent link="base_link"/>
+      <child link="left_wheel"/>
       <origin xyz="0 -${base_width/2} ${z_offset}" rpy="0 0 0"/>
       <axis xyz="0 1 0"/>
@@ -36,5 +44,5 @@
     </joint>
     <!-- left wheel Link -->
-    <link name="${prefix}left_wheel">
+    <link name="left_wheel">
       <collision>
         <origin xyz="0 0 0" rpy="${PI/2} 0 0"/>
@@ -59,7 +67,7 @@
       </inertial>
     </link>
-    <joint name="${prefix}right_wheel_joint" type="continuous">
-      <parent link="${prefix}base_link"/>
-      <child link="${prefix}right_wheel"/>
+    <joint name="right_wheel_joint" type="continuous">
+      <parent link="base_link"/>
+      <child link="right_wheel"/>
       <origin xyz="0 ${base_width/2} ${z_offset}" rpy="0 0 0"/>
       <axis xyz="0 1 0"/>
@@ -67,5 +75,5 @@
     </joint>
     <!-- right wheel Link -->
-    <link name="${prefix}right_wheel">
+    <link name="right_wheel">
       <collision>
         <origin xyz="0 0 0" rpy="${PI/2} 0 0"/>
@@ -90,4 +98,25 @@
       </inertial>
     </link>
+    <!-- sensor links and joints -->
+    <joint name="gps_joint" type="fixed">
+      <parent link="base_link"/>
+      <child link="gps_link"/>
+      <origin xyz="0 0 0" rpy="0 0 0"/>
+    </joint>
+    <link name="gps_link"/>
+    <joint name="scan_joint" type="fixed">
+      <parent link="base_link"/>
+      <child link="base_scan"/>
+      <origin xyz="0 0 0.07" rpy="0 0 0"/>
+    </joint>
+    <link name="base_scan">
+      <visual>
+        <origin xyz="0 0 0" rpy="0 0 0"/>
+        <geometry>
+          <cylinder length="0.05" radius="0.05"/>
+        </geometry>
+        <material name="lidar_color"/>
+      </visual>
+    </link>
   </xacro:macro>
 </robot>

File: asb_webots/resource/asb_webots_robot.urdf (robot description, URDF)
Before this commit: robot asb_webots_robot, 6 links, 5 joints
Links:
- removed link base_footprint
- removed link base_link
- removed link base_scan
- removed link gps_link
- removed link wheel_left_link
- removed link wheel_right_link
Joints:
- removed joint base_joint
- removed joint gps_joint
- removed joint scan_joint
- removed joint wheel_left_joint
- removed joint wheel_right_joint
