Commit message: fixed webots robot and urdf models

File: asb_ros2_control/description/urdf/asb_description.urdf.xacro (robot description, xacro)
@@ -2,121 +2,174 @@
 <robot xmlns:xacro="http://www.ros.org/wiki/xacro">
   <xacro:macro name="asb_description">
-<!--  <xacro:macro name="asb" params="prefix">-->
-    <!-- Constants for robot dimensions -->
-    <xacro:property name="PI" value="3.1415926535897931"/>
-    <xacro:property name="base_mass" value="0.3" /> <!-- arbitrary value for base mass -->
-    <xacro:property name="base_width" value="1.0" />
-    <xacro:property name="base_length" value="2.0" />
-    <xacro:property name="base_height" value="1.5" />
-    <xacro:property name="wheel_mass" value="0.3" /> <!-- arbitrary value for wheel mass -->
-    <xacro:property name="wheel_len" value="0.03" />
-    <xacro:property name="wheel_radius" value="0.15" />
-    <xacro:property name="z_offset" value="-${base_height/2}" /> <!-- Space btw top of beam and each joint -->
-    <!-- Base Link -->
     <link name="base_footprint"/>
     <joint name="base_joint" type="fixed">
         <parent link="base_footprint"/>
         <child link="base_link" />
-        <origin xyz="0 0 0.010" rpy="0 0 0"/>
+        <origin xyz="0 0 0.2" rpy="0 0 0"/>
     </joint>
-    <!-- Base Link -->
+    <!-- BEGIN generated by Webots -->
     <link name="base_link">
+      <visual>
+          <origin xyz="0 0 0.28" rpy="0 0 0"/>
+          <geometry>
+              <box size="1.2 1.5 0.1"/>
+          </geometry>
+      </visual>
       <collision>
-        <origin xyz="0 0 ${base_height/2}" rpy="0 0 0"/>
-        <geometry>
-          <box size="${base_length} ${base_width} ${base_height}"/>
-        </geometry>
+          <origin xyz="0 0 0.28" rpy="0 0 0"/>
+          <geometry>
+              <box size="1.2 1.5 0.1"/>
+          </geometry>
+      </collision>
+    </link>
+    <link name="base_scan_front">
+    </link>
+    <joint name="base_link_base_scan_front_joint" type="fixed">
+      <parent link="base_link"/>
+      <child link="base_scan_front"/>
+      <origin xyz="1.05 0 0.32" rpy="0 0 0"/>
+    </joint>
+    <link name="gnss_link">
+    </link>
+    <joint name="base_link_gnss_link_joint" type="fixed">
+      <parent link="base_link"/>
+      <child link="gnss_link"/>
+      <origin xyz="0.57 0 1.37" rpy="0 0 0"/>
+    </joint>
+    <link name="right_track">
+      <visual>
+          <origin xyz="0 0 -0.0245" rpy="1.570796 0 0"/>
+          <geometry>
+              <box size="1.32 0.351 0.2"/>
+          </geometry>
+      </visual>
+      <collision>
+          <origin xyz="0 0 -0.0245" rpy="1.570796 0 0"/>
+          <geometry>
+              <box size="1.32 0.351 0.2"/>
+          </geometry>
       </collision>
       <visual>
-        <origin xyz="0 0 ${base_height/2}" rpy="0 0 0"/>
-        <geometry>
-          <box size="${base_length} ${base_width} ${base_height}"/>
-        </geometry>
-        <material name="orange"/>
+          <origin xyz="0.844504 0 -0.125681" rpy="1.570808 -0.133483 0"/>
+          <geometry>
+              <box size="0.385 0.1 0.2"/>
+          </geometry>
       </visual>
-    </link>
-    <joint name="left_wheel_joint" type="continuous">
-      <parent link="base_link"/>
-      <child link="left_wheel"/>
-      <origin xyz="0 -${base_width/2} ${z_offset}" rpy="0 0 0"/>
-      <axis xyz="0 1 0"/>
-      <dynamics damping="0.2"/>
-    </joint>
-    <!-- left wheel Link -->
-    <link name="left_wheel">
       <collision>
-        <origin xyz="0 0 0" rpy="${PI/2} 0 0"/>
-        <geometry>
-          <cylinder length="${wheel_len}" radius="${wheel_radius}"/>
-        </geometry>
+          <origin xyz="0.844504 0 -0.125681" rpy="1.570808 -0.133483 0"/>
+          <geometry>
+              <box size="0.385 0.1 0.2"/>
+          </geometry>
       </collision>
       <visual>
-        <origin xyz="0 0 0" rpy="${PI/2} 0 0"/>
-        <geometry>
-          <cylinder length="${wheel_len}" radius="${wheel_radius}"/>
-        </geometry>
-        <material name="black"/>
+          <origin xyz="-0.845 0 -0.126" rpy="1.570805 0.130943 0.000002"/>
+          <geometry>
+              <box size="0.385 0.1 0.2"/>
+          </geometry>
       </visual>
-      <inertial>
-        <origin xyz="0 0 0" rpy="${PI/2} 0 0"/>
-        <mass value="${wheel_mass}"/>
-        <inertia
-                ixx="${wheel_mass / 12.0 * (3*wheel_radius*wheel_radius + wheel_len*wheel_len)}" ixy="0.0" ixz="0.0"
-                iyy="${wheel_mass / 12.0 * (3*wheel_radius*wheel_radius + wheel_len*wheel_len)}" iyz="0.0"
-                izz="${wheel_mass / 2.0 * wheel_radius*wheel_radius}"/>
-      </inertial>
-    </link>
-    <joint name="right_wheel_joint" type="continuous">
-      <parent link="base_link"/>
-      <child link="right_wheel"/>
-      <origin xyz="0 ${base_width/2} ${z_offset}" rpy="0 0 0"/>
-      <axis xyz="0 1 0"/>
-      <dynamics damping="0.2"/>
-    </joint>
-    <!-- right wheel Link -->
-    <link name="right_wheel">
       <collision>
-        <origin xyz="0 0 0" rpy="${PI/2} 0 0"/>
-        <geometry>
-          <cylinder length="${wheel_len}" radius="${wheel_radius}"/>
-        </geometry>
+          <origin xyz="-0.845 0 -0.126" rpy="1.570805 0.130943 0.000002"/>
+          <geometry>
+              <box size="0.385 0.1 0.2"/>
+          </geometry>
       </collision>
       <visual>
-        <origin xyz="0 0 0" rpy="${PI/2} 0 0"/>
-        <geometry>
-          <cylinder length="${wheel_len}" radius="${wheel_radius}"/>
-        </geometry>
-        <material name="black"/>
+          <origin xyz="-1 0 0" rpy="1.5708 0 0"/>
+          <geometry>
+              <cylinder radius="0.151" length="0.2"/>
+          </geometry>
       </visual>
-      <inertial>
-        <origin xyz="0 0 0" rpy="${PI/2} 0 0"/>
-        <mass value="${wheel_mass}"/>
-        <inertia
-                ixx="${wheel_mass / 12.0 * (3*wheel_radius*wheel_radius + wheel_len*wheel_len)}" ixy="0.0" ixz="0.0"
-                iyy="${wheel_mass / 12.0 * (3*wheel_radius*wheel_radius + wheel_len*wheel_len)}" iyz="0.0"
-                izz="${wheel_mass / 2.0 * wheel_radius*wheel_radius}"/>
-      </inertial>
+      <collision>
+          <origin xyz="-1 0 0" rpy="1.5708 0 0"/>
+          <geometry>
+              <cylinder radius="0.151" length="0.2"/>
+          </geometry>
+      </collision>
+      <visual>
+          <origin xyz="1 0 0" rpy="1.5708 0 0"/>
+          <geometry>
+              <cylinder radius="0.151" length="0.2"/>
+          </geometry>
+      </visual>
+      <collision>
+          <origin xyz="1 0 0" rpy="1.5708 0 0"/>
+          <geometry>
+              <cylinder radius="0.151" length="0.2"/>
+          </geometry>
+      </collision>
     </link>
-    <!-- sensor links and joints -->
-    <joint name="gps_joint" type="fixed">
+    <joint name="base_link_right_track_joint" type="fixed">
       <parent link="base_link"/>
-      <child link="gps_link"/>
-      <origin xyz="0 0 0" rpy="0 0 0"/>
+      <child link="right_track"/>
+      <origin xyz="0 -0.5 0" rpy="0 0 0"/>
     </joint>
-    <link name="gps_link"/>
-    <joint name="scan_joint" type="fixed">
+    <link name="left_track">
+      <visual>
+          <origin xyz="0 0 -0.0245" rpy="1.570796 0 0"/>
+          <geometry>
+              <box size="1.32 0.351 0.2"/>
+          </geometry>
+      </visual>
+      <collision>
+          <origin xyz="0 0 -0.0245" rpy="1.570796 0 0"/>
+          <geometry>
+              <box size="1.32 0.351 0.2"/>
+          </geometry>
+      </collision>
+      <visual>
+          <origin xyz="0.844504 0 -0.125681" rpy="1.570808 -0.133483 0"/>
+          <geometry>
+              <box size="0.385 0.1 0.2"/>
+          </geometry>
+      </visual>
+      <collision>
+          <origin xyz="0.844504 0 -0.125681" rpy="1.570808 -0.133483 0"/>
+          <geometry>
+              <box size="0.385 0.1 0.2"/>
+          </geometry>
+      </collision>
+      <visual>
+          <origin xyz="-0.845 0 -0.126" rpy="1.570805 0.130943 0.000002"/>
+          <geometry>
+              <box size="0.385 0.1 0.2"/>
+          </geometry>
+      </visual>
+      <collision>
+          <origin xyz="-0.845 0 -0.126" rpy="1.570805 0.130943 0.000002"/>
+          <geometry>
+              <box size="0.385 0.1 0.2"/>
+          </geometry>
+      </collision>
+      <visual>
+          <origin xyz="-1 0 0" rpy="1.5708 0 0"/>
+          <geometry>
+              <cylinder radius="0.151" length="0.2"/>
+          </geometry>
+      </visual>
+      <collision>
+          <origin xyz="-1 0 0" rpy="1.5708 0 0"/>
+          <geometry>
+              <cylinder radius="0.151" length="0.2"/>
+          </geometry>
+      </collision>
+      <visual>
+          <origin xyz="1 0 0" rpy="1.5708 0 0"/>
+          <geometry>
+              <cylinder radius="0.151" length="0.2"/>
+          </geometry>
+      </visual>
+      <collision>
+          <origin xyz="1 0 0" rpy="1.5708 0 0"/>
+          <geometry>
+              <cylinder radius="0.151" length="0.2"/>
+          </geometry>
+      </collision>
+    </link>
+    <joint name="base_link_left_track_joint" type="fixed">
       <parent link="base_link"/>
-      <child link="base_scan"/>
-      <origin xyz="0 0 0.07" rpy="0 0 0"/>
+      <child link="left_track"/>
+      <origin xyz="0 0.5 0" rpy="0 0 0"/>
     </joint>
-    <link name="base_scan">
-      <visual>
-        <origin xyz="0 0 0" rpy="0 0 0"/>
-        <geometry>
-          <cylinder length="0.05" radius="0.05"/>
-        </geometry>
-        <material name="lidar_color"/>
-      </visual>
-    </link>
+    <!-- END generated by Webots -->
   </xacro:macro>
 </robot>

Commit message: added second gnss sensor, fixed webots gnss sensor in driver

File: asb_ros2_control/description/urdf/asb_description.urdf.xacro (robot description, xacro)
@@ -11,14 +11,14 @@
     <link name="base_link">
       <visual>
-          <origin xyz="0 0 0.28" rpy="0 0 0"/>
-          <geometry>
-              <box size="1.2 1.5 0.1"/>
-          </geometry>
+        <origin xyz="0 0 0.28" rpy="0 0 0"/>
+        <geometry>
+          <box size="1.2 1.5 0.1"/>
+        </geometry>
       </visual>
       <collision>
-          <origin xyz="0 0 0.28" rpy="0 0 0"/>
-          <geometry>
-              <box size="1.2 1.5 0.1"/>
-          </geometry>
+        <origin xyz="0 0 0.28" rpy="0 0 0"/>
+        <geometry>
+          <box size="1.2 1.5 0.1"/>
+        </geometry>
       </collision>
     </link>
@@ -29,4 +29,11 @@
       <child link="base_scan_front"/>
       <origin xyz="1.05 0 0.32" rpy="0 0 0"/>
+    </joint>
+    <link name="gnss_link_2">
+    </link>
+    <joint name="base_link_gnss_link_2_joint" type="fixed">
+      <parent link="base_link"/>
+      <child link="gnss_link_2"/>
+      <origin xyz="-0.57 0 1.37" rpy="0 0 0"/>
     </joint>
     <link name="gnss_link">
@@ -39,62 +46,62 @@
     <link name="right_track">
       <visual>
-          <origin xyz="0 0 -0.0245" rpy="1.570796 0 0"/>
-          <geometry>
-              <box size="1.32 0.351 0.2"/>
-          </geometry>
+        <origin xyz="0 0 -0.0245" rpy="1.570796 0 0"/>
+        <geometry>
+          <box size="1.32 0.351 0.2"/>
+        </geometry>
       </visual>
       <collision>
-          <origin xyz="0 0 -0.0245" rpy="1.570796 0 0"/>
-          <geometry>
-              <box size="1.32 0.351 0.2"/>
-          </geometry>
+        <origin xyz="0 0 -0.0245" rpy="1.570796 0 0"/>
+        <geometry>
+          <box size="1.32 0.351 0.2"/>
+        </geometry>
       </collision>
       <visual>
-          <origin xyz="0.844504 0 -0.125681" rpy="1.570808 -0.133483 0"/>
-          <geometry>
-              <box size="0.385 0.1 0.2"/>
-          </geometry>
+        <origin xyz="0.844504 0 -0.125681" rpy="1.570808 -0.133483 0"/>
+        <geometry>
+          <box size="0.385 0.1 0.2"/>
+        </geometry>
       </visual>
       <collision>
-          <origin xyz="0.844504 0 -0.125681" rpy="1.570808 -0.133483 0"/>
-          <geometry>
-              <box size="0.385 0.1 0.2"/>
-          </geometry>
+        <origin xyz="0.844504 0 -0.125681" rpy="1.570808 -0.133483 0"/>
+        <geometry>
+          <box size="0.385 0.1 0.2"/>
+        </geometry>
       </collision>
       <visual>
-          <origin xyz="-0.845 0 -0.126" rpy="1.570805 0.130943 0.000002"/>
-          <geometry>
-              <box size="0.385 0.1 0.2"/>
-          </geometry>
+        <origin xyz="-0.845 0 -0.126" rpy="1.570805 0.130943 0.000002"/>
+        <geometry>
+          <box size="0.385 0.1 0.2"/>
+        </geometry>
       </visual>
       <collision>
-          <origin xyz="-0.845 0 -0.126" rpy="1.570805 0.130943 0.000002"/>
-          <geometry>
-              <box size="0.385 0.1 0.2"/>
-          </geometry>
+        <origin xyz="-0.845 0 -0.126" rpy="1.570805 0.130943 0.000002"/>
+        <geometry>
+          <box size="0.385 0.1 0.2"/>
+        </geometry>
       </collision>
       <visual>
-          <origin xyz="-1 0 0" rpy="1.5708 0 0"/>
-          <geometry>
-              <cylinder radius="0.151" length="0.2"/>
-          </geometry>
+        <origin xyz="-1 0 0" rpy="1.5708 0 0"/>
+        <geometry>
+          <cylinder radius="0.151" length="0.2"/>
+        </geometry>
       </visual>
       <collision>
-          <origin xyz="-1 0 0" rpy="1.5708 0 0"/>
-          <geometry>
-              <cylinder radius="0.151" length="0.2"/>
-          </geometry>
+        <origin xyz="-1 0 0" rpy="1.5708 0 0"/>
+        <geometry>
+          <cylinder radius="0.151" length="0.2"/>
+        </geometry>
       </collision>
       <visual>
-          <origin xyz="1 0 0" rpy="1.5708 0 0"/>
-          <geometry>
-              <cylinder radius="0.151" length="0.2"/>
-          </geometry>
+        <origin xyz="1 0 0" rpy="1.5708 0 0"/>
+        <geometry>
+          <cylinder radius="0.151" length="0.2"/>
+        </geometry>
       </visual>
       <collision>
-          <origin xyz="1 0 0" rpy="1.5708 0 0"/>
-          <geometry>
-              <cylinder radius="0.151" length="0.2"/>
-          </geometry>
+        <origin xyz="1 0 0" rpy="1.5708 0 0"/>
+        <geometry>
+          <cylinder radius="0.151" length="0.2"/>
+        </geometry>
       </collision>
     </link>
@@ -106,62 +113,62 @@
     <link name="left_track">
       <visual>
-          <origin xyz="0 0 -0.0245" rpy="1.570796 0 0"/>
-          <geometry>
-              <box size="1.32 0.351 0.2"/>
-          </geometry>
+        <origin xyz="0 0 -0.0245" rpy="1.570796 0 0"/>
+        <geometry>
+          <box size="1.32 0.351 0.2"/>
+        </geometry>
       </visual>
       <collision>
-          <origin xyz="0 0 -0.0245" rpy="1.570796 0 0"/>
-          <geometry>
-              <box size="1.32 0.351 0.2"/>
-          </geometry>
+        <origin xyz="0 0 -0.0245" rpy="1.570796 0 0"/>
+        <geometry>
+          <box size="1.32 0.351 0.2"/>
+        </geometry>
       </collision>
       <visual>
-          <origin xyz="0.844504 0 -0.125681" rpy="1.570808 -0.133483 0"/>
-          <geometry>
-              <box size="0.385 0.1 0.2"/>
-          </geometry>
+        <origin xyz="0.844504 0 -0.125681" rpy="1.570808 -0.133483 0"/>
+        <geometry>
+          <box size="0.385 0.1 0.2"/>
+        </geometry>
       </visual>
       <collision>
-          <origin xyz="0.844504 0 -0.125681" rpy="1.570808 -0.133483 0"/>
-          <geometry>
-              <box size="0.385 0.1 0.2"/>
-          </geometry>
+        <origin xyz="0.844504 0 -0.125681" rpy="1.570808 -0.133483 0"/>
+        <geometry>
+          <box size="0.385 0.1 0.2"/>
+        </geometry>
       </collision>
       <visual>
-          <origin xyz="-0.845 0 -0.126" rpy="1.570805 0.130943 0.000002"/>
-          <geometry>
-              <box size="0.385 0.1 0.2"/>
-          </geometry>
+        <origin xyz="-0.845 0 -0.126" rpy="1.570805 0.130943 0.000002"/>
+        <geometry>
+          <box size="0.385 0.1 0.2"/>
+        </geometry>
       </visual>
       <collision>
-          <origin xyz="-0.845 0 -0.126" rpy="1.570805 0.130943 0.000002"/>
-          <geometry>
-              <box size="0.385 0.1 0.2"/>
-          </geometry>
+        <origin xyz="-0.845 0 -0.126" rpy="1.570805 0.130943 0.000002"/>
+        <geometry>
+          <box size="0.385 0.1 0.2"/>
+        </geometry>
       </collision>
       <visual>
-          <origin xyz="-1 0 0" rpy="1.5708 0 0"/>
-          <geometry>
-              <cylinder radius="0.151" length="0.2"/>
-          </geometry>
+        <origin xyz="-1 0 0" rpy="1.5708 0 0"/>
+        <geometry>
+          <cylinder radius="0.151" length="0.2"/>
+        </geometry>
       </visual>
       <collision>
-          <origin xyz="-1 0 0" rpy="1.5708 0 0"/>
-          <geometry>
-              <cylinder radius="0.151" length="0.2"/>
-          </geometry>
+        <origin xyz="-1 0 0" rpy="1.5708 0 0"/>
+        <geometry>
+          <cylinder radius="0.151" length="0.2"/>
+        </geometry>
       </collision>
       <visual>
-          <origin xyz="1 0 0" rpy="1.5708 0 0"/>
-          <geometry>
-              <cylinder radius="0.151" length="0.2"/>
-          </geometry>
+        <origin xyz="1 0 0" rpy="1.5708 0 0"/>
+        <geometry>
+          <cylinder radius="0.151" length="0.2"/>
+        </geometry>
       </visual>
       <collision>
-          <origin xyz="1 0 0" rpy="1.5708 0 0"/>
-          <geometry>
-              <cylinder radius="0.151" length="0.2"/>
-          </geometry>
+        <origin xyz="1 0 0" rpy="1.5708 0 0"/>
+        <geometry>
+          <cylinder radius="0.151" length="0.2"/>
+        </geometry>
       </collision>
     </link>

Commit message: tuned ekf and nav2 params, added rear LIDAR

File: asb_ros2_control/description/urdf/asb_description.urdf.xacro (robot description, xacro)
@@ -23,4 +23,11 @@
       </collision>
     </link>
+    <link name="base_scan_rear">
+    </link>
+    <joint name="base_link_base_scan_rear_joint" type="fixed">
+      <parent link="base_link"/>
+      <child link="base_scan_rear"/>
+      <origin xyz="-1.05 0 0.32" rpy="0 0 3.14159"/>
+    </joint>
     <link name="base_scan_front">
     </link>

Commit message: added gyro sensor

File: asb_ros2_control/description/urdf/asb_description.urdf.xacro (robot description, xacro)
@@ -37,4 +37,32 @@
       <origin xyz="1.05 0 0.32" rpy="0 0 0"/>
     </joint>
+    <link name="imu_link">
+    </link>
+    <joint name="base_link_imu_link_joint" type="fixed">
+      <parent link="base_link"/>
+      <child link="imu_link"/>
+      <origin xyz="0 0 0.23" rpy="0 0 0"/>
+    </joint>
+    <link name="inertial_link">
+    </link>
+    <joint name="imu_link_inertial_link_joint" type="fixed">
+      <parent link="imu_link"/>
+      <child link="inertial_link"/>
+      <origin xyz="0 0 0" rpy="0 0 0"/>
+    </joint>
+    <link name="gyro_link">
+    </link>
+    <joint name="imu_link_gyro_link_joint" type="fixed">
+      <parent link="imu_link"/>
+      <child link="gyro_link"/>
+      <origin xyz="0 0 0" rpy="0 0 0"/>
+    </joint>
+    <link name="accelerometer_link">
+    </link>
+    <joint name="imu_link_accelerometer_link_joint" type="fixed">
+      <parent link="imu_link"/>
+      <child link="accelerometer_link"/>
+      <origin xyz="0 0 0" rpy="0 0 0"/>
+    </joint>
     <link name="gnss_link_2">
     </link>
