Commit message: added Ouster OS0-32 and improved urdf robot description

File: asb_ros2_control/description/urdf/asb_description.urdf.xacro (robot description, xacro)
@@ -22,5 +22,79 @@
         </geometry>
       </collision>
-    </link>
+      <visual>
+        <origin xyz="0 0.6 0.53" rpy="0 0 0"/>
+        <geometry>
+          <box size="1.5 0.2 0.4"/>
+        </geometry>
+      </visual>
+      <collision>
+        <origin xyz="0 0.6 0.53" rpy="0 0 0"/>
+        <geometry>
+          <box size="1.5 0.2 0.4"/>
+        </geometry>
+      </collision>
+      <visual>
+        <origin xyz="0 -0.6 0.53" rpy="0 0 0"/>
+        <geometry>
+          <box size="1.5 0.2 0.4"/>
+        </geometry>
+      </visual>
+      <collision>
+        <origin xyz="0 -0.6 0.53" rpy="0 0 0"/>
+        <geometry>
+          <box size="1.5 0.2 0.4"/>
+        </geometry>
+      </collision>
+      <visual>
+        <origin xyz="0 0 0.83" rpy="0 0 0"/>
+        <geometry>
+          <box size="1.5 0.9 1"/>
+        </geometry>
+      </visual>
+      <collision>
+        <origin xyz="0 0 0.83" rpy="0 0 0"/>
+        <geometry>
+          <box size="1.5 0.9 1"/>
+        </geometry>
+      </collision>
+    </link>
+    <link name="base_scan_rear_left">
+      <visual>
+        <origin xyz="0 0 0" rpy="0 0 0"/>
+        <geometry>
+          <cylinder radius="0.0435" length="0.0742"/>
+        </geometry>
+      </visual>
+      <collision>
+        <origin xyz="0 0 0" rpy="0 0 0"/>
+        <geometry>
+          <cylinder radius="0.0435" length="0.0742"/>
+        </geometry>
+      </collision>
+    </link>
+    <joint name="base_link_base_scan_rear_left_joint" type="fixed">
+      <parent link="base_link"/>
+      <child link="base_scan_rear_left"/>
+      <origin xyz="-1.18 0.76 0.52" rpy="0 0 2.356194"/>
+    </joint>
+    <link name="base_scan_front_right">
+      <visual>
+        <origin xyz="0 0 0" rpy="0 0 0"/>
+        <geometry>
+          <cylinder radius="0.0435" length="0.0742"/>
+        </geometry>
+      </visual>
+      <collision>
+        <origin xyz="0 0 0" rpy="0 0 0"/>
+        <geometry>
+          <cylinder radius="0.0435" length="0.0742"/>
+        </geometry>
+      </collision>
+    </link>
+    <joint name="base_link_base_scan_front_right_joint" type="fixed">
+      <parent link="base_link"/>
+      <child link="base_scan_front_right"/>
+      <origin xyz="1.18 -0.76 0.52" rpy="0 0 -0.785398"/>
+    </joint>
     <link name="base_scan_rear">
     </link>
@@ -65,11 +139,4 @@
       <origin xyz="0 0 0" rpy="0 0 0"/>
     </joint>
-    <link name="gnss_link_2">
-    </link>
-    <joint name="base_link_gnss_link_2_joint" type="fixed">
-      <parent link="base_link"/>
-      <child link="gnss_link_2"/>
-      <origin xyz="-0.57 0 1.37" rpy="0 0 0"/>
-    </joint>
     <link name="gnss_link">
     </link>
@@ -81,4 +148,16 @@
     <link name="right_track">
       <visual>
+        <origin xyz="0 0 0.1" rpy="1.570796 0 0"/>
+        <geometry>
+          <box size="2 0.1 0.2"/>
+        </geometry>
+      </visual>
+      <collision>
+        <origin xyz="0 0 0.1" rpy="1.570796 0 0"/>
+        <geometry>
+          <box size="2 0.1 0.2"/>
+        </geometry>
+      </collision>
+      <visual>
         <origin xyz="0 0 -0.0245" rpy="1.570796 0 0"/>
         <geometry>
@@ -147,4 +226,16 @@
     </joint>
     <link name="left_track">
+      <visual>
+        <origin xyz="0 0 0.1" rpy="1.570796 0 0"/>
+        <geometry>
+          <box size="2 0.1 0.2"/>
+        </geometry>
+      </visual>
+      <collision>
+        <origin xyz="0 0 0.1" rpy="1.570796 0 0"/>
+        <geometry>
+          <box size="2 0.1 0.2"/>
+        </geometry>
+      </collision>
       <visual>
         <origin xyz="0 0 -0.0245" rpy="1.570796 0 0"/>

Commit message: improved webots Ouster OS0 and fixed single layer lidars

File: asb_ros2_control/description/urdf/asb_description.urdf.xacro (robot description, xacro)
@@ -59,15 +59,53 @@
       </collision>
     </link>
+    <link name="base_scan_rear_left_multilayer">
+      <visual>
+        <origin xyz="0 0 0" rpy="0 0 0"/>
+        <geometry>
+          <cylinder radius="0.0435" length="0.0742"/>
+        </geometry>
+      </visual>
+      <collision>
+        <origin xyz="0 0 0" rpy="0 0 0"/>
+        <geometry>
+          <cylinder radius="0.0435" length="0.0742"/>
+        </geometry>
+      </collision>
+    </link>
+    <joint name="base_link_base_scan_rear_left_multilayer_joint" type="fixed">
+      <parent link="base_link"/>
+      <child link="base_scan_rear_left_multilayer"/>
+      <origin xyz="-1.18 0.76 0.4" rpy="0 0 2.356194"/>
+    </joint>
+    <link name="base_scan_front_right_multilayer">
+      <visual>
+        <origin xyz="0 0 0" rpy="0 0 0"/>
+        <geometry>
+          <cylinder radius="0.0435" length="0.0742"/>
+        </geometry>
+      </visual>
+      <collision>
+        <origin xyz="0 0 0" rpy="0 0 0"/>
+        <geometry>
+          <cylinder radius="0.0435" length="0.0742"/>
+        </geometry>
+      </collision>
+    </link>
+    <joint name="base_link_base_scan_front_right_multilayer_joint" type="fixed">
+      <parent link="base_link"/>
+      <child link="base_scan_front_right_multilayer"/>
+      <origin xyz="1.18 -0.76 0.4" rpy="0 0 -0.785398"/>
+    </joint>
     <link name="base_scan_rear_left">
       <visual>
-        <origin xyz="0 0 0" rpy="0 0 0"/>
-        <geometry>
-          <cylinder radius="0.0435" length="0.0742"/>
-        </geometry>
-      </visual>
-      <collision>
-        <origin xyz="0 0 0" rpy="0 0 0"/>
-        <geometry>
-          <cylinder radius="0.0435" length="0.0742"/>
+        <origin xyz="0 0 -0.011" rpy="1.570741 0.000118 -1.570741"/>
+        <geometry>
+          <box size="0.06 0.087 0.06"/>
+        </geometry>
+      </visual>
+      <collision>
+        <origin xyz="0 0 -0.011" rpy="1.570741 0.000118 -1.570741"/>
+        <geometry>
+          <box size="0.06 0.087 0.06"/>
         </geometry>
       </collision>
@@ -76,17 +114,17 @@
       <parent link="base_link"/>
       <child link="base_scan_rear_left"/>
-      <origin xyz="-1.18 0.76 0.52" rpy="0 0 2.356194"/>
+      <origin xyz="-1.18 0.76 0.3" rpy="0 0 2.356194"/>
     </joint>
     <link name="base_scan_front_right">
       <visual>
-        <origin xyz="0 0 0" rpy="0 0 0"/>
-        <geometry>
-          <cylinder radius="0.0435" length="0.0742"/>
-        </geometry>
-      </visual>
-      <collision>
-        <origin xyz="0 0 0" rpy="0 0 0"/>
-        <geometry>
-          <cylinder radius="0.0435" length="0.0742"/>
+        <origin xyz="0 0 -0.011" rpy="1.570741 0.000118 -1.570741"/>
+        <geometry>
+          <box size="0.06 0.087 0.06"/>
+        </geometry>
+      </visual>
+      <collision>
+        <origin xyz="0 0 -0.011" rpy="1.570741 0.000118 -1.570741"/>
+        <geometry>
+          <box size="0.06 0.087 0.06"/>
         </geometry>
       </collision>
@@ -95,19 +133,5 @@
       <parent link="base_link"/>
       <child link="base_scan_front_right"/>
-      <origin xyz="1.18 -0.76 0.52" rpy="0 0 -0.785398"/>
-    </joint>
-    <link name="base_scan_rear">
-    </link>
-    <joint name="base_link_base_scan_rear_joint" type="fixed">
-      <parent link="base_link"/>
-      <child link="base_scan_rear"/>
-      <origin xyz="-1.05 0 0.32" rpy="0 0 3.14159"/>
-    </joint>
-    <link name="base_scan_front">
-    </link>
-    <joint name="base_link_base_scan_front_joint" type="fixed">
-      <parent link="base_link"/>
-      <child link="base_scan_front"/>
-      <origin xyz="1.05 0 0.32" rpy="0 0 0"/>
+      <origin xyz="1.18 -0.76 0.3" rpy="0 0 -0.785398"/>
     </joint>
     <link name="imu_link">

Commit message: improved approximate webots and URDF robot dimensions

File: asb_ros2_control/description/urdf/asb_description.urdf.xacro (robot description, xacro)
@@ -11,52 +11,522 @@
     <link name="base_link">
       <visual>
-        <origin xyz="0 0 0.28" rpy="0 0 0"/>
-        <geometry>
-          <box size="1.2 1.5 0.1"/>
-        </geometry>
-      </visual>
-      <collision>
-        <origin xyz="0 0 0.28" rpy="0 0 0"/>
-        <geometry>
-          <box size="1.2 1.5 0.1"/>
-        </geometry>
-      </collision>
-      <visual>
-        <origin xyz="0 0.6 0.53" rpy="0 0 0"/>
-        <geometry>
-          <box size="1.5 0.2 0.4"/>
-        </geometry>
-      </visual>
-      <collision>
-        <origin xyz="0 0.6 0.53" rpy="0 0 0"/>
-        <geometry>
-          <box size="1.5 0.2 0.4"/>
-        </geometry>
-      </collision>
-      <visual>
-        <origin xyz="0 -0.6 0.53" rpy="0 0 0"/>
-        <geometry>
-          <box size="1.5 0.2 0.4"/>
-        </geometry>
-      </visual>
-      <collision>
-        <origin xyz="0 -0.6 0.53" rpy="0 0 0"/>
-        <geometry>
-          <box size="1.5 0.2 0.4"/>
-        </geometry>
-      </collision>
-      <visual>
-        <origin xyz="0 0 0.83" rpy="0 0 0"/>
-        <geometry>
-          <box size="1.5 0.9 1"/>
-        </geometry>
-      </visual>
-      <collision>
-        <origin xyz="0 0 0.83" rpy="0 0 0"/>
-        <geometry>
-          <box size="1.5 0.9 1"/>
-        </geometry>
-      </collision>
-    </link>
+        <origin xyz="0.491 0 0.315" rpy="0 0 0"/>
+        <geometry>
+          <box size="0.12 1.48 0.12"/>
+        </geometry>
+      </visual>
+      <collision>
+        <origin xyz="0.491 0 0.315" rpy="0 0 0"/>
+        <geometry>
+          <box size="0.12 1.48 0.12"/>
+        </geometry>
+      </collision>
+      <visual>
+        <origin xyz="0.491 0.745 0.315" rpy="0 0 0"/>
+        <geometry>
+          <box size="0.14 0.01 0.14"/>
+        </geometry>
+      </visual>
+      <collision>
+        <origin xyz="0.491 0.745 0.315" rpy="0 0 0"/>
+        <geometry>
+          <box size="0.14 0.01 0.14"/>
+        </geometry>
+      </collision>
+      <visual>
+        <origin xyz="0.491 0.635 0.135" rpy="0 0 0"/>
+        <geometry>
+          <box size="0.12 0.07 0.24"/>
+        </geometry>
+      </visual>
+      <collision>
+        <origin xyz="0.491 0.635 0.135" rpy="0 0 0"/>
+        <geometry>
+          <box size="0.12 0.07 0.24"/>
+        </geometry>
+      </collision>
+      <visual>
+        <origin xyz="0.491 0.6135 0.008" rpy="-0.7854 0 0"/>
+        <geometry>
+          <box size="0.121 0.07 0.09"/>
+        </geometry>
+      </visual>
+      <collision>
+        <origin xyz="0.491 0.6135 0.008" rpy="-0.7854 0 0"/>
+        <geometry>
+          <box size="0.121 0.07 0.09"/>
+        </geometry>
+      </collision>
+      <visual>
+        <origin xyz="0.491 0.5714 -0.0134" rpy="0 0 0"/>
+        <geometry>
+          <box size="0.12 0.07 0.07"/>
+        </geometry>
+      </visual>
+      <collision>
+        <origin xyz="0.491 0.5714 -0.0134" rpy="0 0 0"/>
+        <geometry>
+          <box size="0.12 0.07 0.07"/>
+        </geometry>
+      </collision>
+      <visual>
+        <origin xyz="0.491 -0.745 0.315" rpy="0 0 0"/>
+        <geometry>
+          <box size="0.14 0.01 0.14"/>
+        </geometry>
+      </visual>
+      <collision>
+        <origin xyz="0.491 -0.745 0.315" rpy="0 0 0"/>
+        <geometry>
+          <box size="0.14 0.01 0.14"/>
+        </geometry>
+      </collision>
+      <visual>
+        <origin xyz="0.491 -0.635 0.135" rpy="0 0 0"/>
+        <geometry>
+          <box size="0.12 0.07 0.24"/>
+        </geometry>
+      </visual>
+      <collision>
+        <origin xyz="0.491 -0.635 0.135" rpy="0 0 0"/>
+        <geometry>
+          <box size="0.12 0.07 0.24"/>
+        </geometry>
+      </collision>
+      <visual>
+        <origin xyz="0.491 -0.6135 0.008" rpy="0.7854 0 0"/>
+        <geometry>
+          <box size="0.121 0.07 0.09"/>
+        </geometry>
+      </visual>
+      <collision>
+        <origin xyz="0.491 -0.6135 0.008" rpy="0.7854 0 0"/>
+        <geometry>
+          <box size="0.121 0.07 0.09"/>
+        </geometry>
+      </collision>
+      <visual>
+        <origin xyz="0.491 -0.5714 -0.0134" rpy="0 0 0"/>
+        <geometry>
+          <box size="0.12 0.07 0.07"/>
+        </geometry>
+      </visual>
+      <collision>
+        <origin xyz="0.491 -0.5714 -0.0134" rpy="0 0 0"/>
+        <geometry>
+          <box size="0.12 0.07 0.07"/>
+        </geometry>
+      </collision>
+      <visual>
+        <origin xyz="-0.106 0 0.315" rpy="0 0 0"/>
+        <geometry>
+          <box size="0.12 1.48 0.12"/>
+        </geometry>
+      </visual>
+      <collision>
+        <origin xyz="-0.106 0 0.315" rpy="0 0 0"/>
+        <geometry>
+          <box size="0.12 1.48 0.12"/>
+        </geometry>
+      </collision>
+      <visual>
+        <origin xyz="-0.106 0.745 0.315" rpy="0 0 0"/>
+        <geometry>
+          <box size="0.14 0.01 0.14"/>
+        </geometry>
+      </visual>
+      <collision>
+        <origin xyz="-0.106 0.745 0.315" rpy="0 0 0"/>
+        <geometry>
+          <box size="0.14 0.01 0.14"/>
+        </geometry>
+      </collision>
+      <visual>
+        <origin xyz="-0.106 0.635 0.135" rpy="0 0 0"/>
+        <geometry>
+          <box size="0.12 0.07 0.24"/>
+        </geometry>
+      </visual>
+      <collision>
+        <origin xyz="-0.106 0.635 0.135" rpy="0 0 0"/>
+        <geometry>
+          <box size="0.12 0.07 0.24"/>
+        </geometry>
+      </collision>
+      <visual>
+        <origin xyz="-0.106 0.6135 0.008" rpy="-0.7854 0 0"/>
+        <geometry>
+          <box size="0.121 0.07 0.09"/>
+        </geometry>
+      </visual>
+      <collision>
+        <origin xyz="-0.106 0.6135 0.008" rpy="-0.7854 0 0"/>
+        <geometry>
+          <box size="0.121 0.07 0.09"/>
+        </geometry>
+      </collision>
+      <visual>
+        <origin xyz="-0.106 0.5714 -0.0134" rpy="0 0 0"/>
+        <geometry>
+          <box size="0.12 0.07 0.07"/>
+        </geometry>
+      </visual>
+      <collision>
+        <origin xyz="-0.106 0.5714 -0.0134" rpy="0 0 0"/>
+        <geometry>
+          <box size="0.12 0.07 0.07"/>
+        </geometry>
+      </collision>
+      <visual>
+        <origin xyz="-0.106 -0.745 0.315" rpy="0 0 0"/>
+        <geometry>
+          <box size="0.14 0.01 0.14"/>
+        </geometry>
+      </visual>
+      <collision>
+        <origin xyz="-0.106 -0.745 0.315" rpy="0 0 0"/>
+        <geometry>
+          <box size="0.14 0.01 0.14"/>
+        </geometry>
+      </collision>
+      <visual>
+        <origin xyz="-0.106 -0.635 0.135" rpy="0 0 0"/>
+        <geometry>
+          <box size="0.12 0.07 0.24"/>
+        </geometry>
+      </visual>
+      <collision>
+        <origin xyz="-0.106 -0.635 0.135" rpy="0 0 0"/>
+        <geometry>
+          <box size="0.12 0.07 0.24"/>
+        </geometry>
+      </collision>
+      <visual>
+        <origin xyz="-0.106 -0.6135 0.008" rpy="-0.7854 0 0"/>
+        <geometry>
+          <box size="0.121 0.07 0.09"/>
+        </geometry>
+      </visual>
+      <collision>
+        <origin xyz="-0.106 -0.6135 0.008" rpy="-0.7854 0 0"/>
+        <geometry>
+          <box size="0.121 0.07 0.09"/>
+        </geometry>
+      </collision>
+      <visual>
+        <origin xyz="-0.106 -0.5714 -0.0134" rpy="0 0 0"/>
+        <geometry>
+          <box size="0.12 0.07 0.07"/>
+        </geometry>
+      </visual>
+      <collision>
+        <origin xyz="-0.106 -0.5714 -0.0134" rpy="0 0 0"/>
+        <geometry>
+          <box size="0.12 0.07 0.07"/>
+        </geometry>
+      </collision>
+      <visual>
+        <origin xyz="-0.491 0 0.315" rpy="0 0 0"/>
+        <geometry>
+          <box size="0.12 1.48 0.12"/>
+        </geometry>
+      </visual>
+      <collision>
+        <origin xyz="-0.491 0 0.315" rpy="0 0 0"/>
+        <geometry>
+          <box size="0.12 1.48 0.12"/>
+        </geometry>
+      </collision>
+      <visual>
+        <origin xyz="-0.491 0.745 0.315" rpy="0 0 0"/>
+        <geometry>
+          <box size="0.14 0.01 0.14"/>
+        </geometry>
+      </visual>
+      <collision>
+        <origin xyz="-0.491 0.745 0.315" rpy="0 0 0"/>
+        <geometry>
+          <box size="0.14 0.01 0.14"/>
+        </geometry>
+      </collision>
+      <visual>
+        <origin xyz="-0.491 0.635 0.135" rpy="0 0 0"/>
+        <geometry>
+          <box size="0.12 0.07 0.24"/>
+        </geometry>
+      </visual>
+      <collision>
+        <origin xyz="-0.491 0.635 0.135" rpy="0 0 0"/>
+        <geometry>
+          <box size="0.12 0.07 0.24"/>
+        </geometry>
+      </collision>
+      <visual>
+        <origin xyz="-0.491 0.6135 0.008" rpy="-0.7854 0 0"/>
+        <geometry>
+          <box size="0.121 0.07 0.09"/>
+        </geometry>
+      </visual>
+      <collision>
+        <origin xyz="-0.491 0.6135 0.008" rpy="-0.7854 0 0"/>
+        <geometry>
+          <box size="0.121 0.07 0.09"/>
+        </geometry>
+      </collision>
+      <visual>
+        <origin xyz="-0.491 0.5714 -0.0134" rpy="0 0 0"/>
+        <geometry>
+          <box size="0.12 0.07 0.07"/>
+        </geometry>
+      </visual>
+      <collision>
+        <origin xyz="-0.491 0.5714 -0.0134" rpy="0 0 0"/>
+        <geometry>
+          <box size="0.12 0.07 0.07"/>
+        </geometry>
+      </collision>
+      <visual>
+        <origin xyz="-0.491 -0.745 0.315" rpy="0 0 0"/>
+        <geometry>
+          <box size="0.14 0.01 0.14"/>
+        </geometry>
+      </visual>
+      <collision>
+        <origin xyz="-0.491 -0.745 0.315" rpy="0 0 0"/>
+        <geometry>
+          <box size="0.14 0.01 0.14"/>
+        </geometry>
+      </collision>
+      <visual>
+        <origin xyz="-0.491 -0.635 0.135" rpy="0 0 0"/>
+        <geometry>
+          <box size="0.12 0.07 0.24"/>
+        </geometry>
+      </visual>
+      <collision>
+        <origin xyz="-0.491 -0.635 0.135" rpy="0 0 0"/>
+        <geometry>
+          <box size="0.12 0.07 0.24"/>
+        </geometry>
+      </collision>
+      <visual>
+        <origin xyz="-0.491 -0.6135 0.008" rpy="-0.7854 0 0"/>
+        <geometry>
+          <box size="0.121 0.07 0.09"/>
+        </geometry>
+      </visual>
+      <collision>
+        <origin xyz="-0.491 -0.6135 0.008" rpy="-0.7854 0 0"/>
+        <geometry>
+          <box size="0.121 0.07 0.09"/>
+        </geometry>
+      </collision>
+      <visual>
+        <origin xyz="-0.491 -0.5714 -0.0134" rpy="0 0 0"/>
+        <geometry>
+          <box size="0.12 0.07 0.07"/>
+        </geometry>
+      </visual>
+      <collision>
+        <origin xyz="-0.491 -0.5714 -0.0134" rpy="0 0 0"/>
+        <geometry>
+          <box size="0.12 0.07 0.07"/>
+        </geometry>
+      </collision>
+      <visual>
+        <origin xyz="0 0.6 0.59" rpy="0 0 0"/>
+        <geometry>
+          <box size="1.3 0.205 0.425"/>
+        </geometry>
+      </visual>
+      <collision>
+        <origin xyz="0 0.6 0.59" rpy="0 0 0"/>
+        <geometry>
+          <box size="1.3 0.205 0.425"/>
+        </geometry>
+      </collision>
+      <visual>
+        <origin xyz="0 -0.6 0.59" rpy="0 0 0"/>
+        <geometry>
+          <box size="1.3 0.205 0.425"/>
+        </geometry>
+      </visual>
+      <collision>
+        <origin xyz="0 -0.6 0.59" rpy="0 0 0"/>
+        <geometry>
+          <box size="1.3 0.205 0.425"/>
+        </geometry>
+      </collision>
+      <visual>
+        <origin xyz="-0.15 0 0.88" rpy="0 0 0"/>
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
Commit message: fixed imu and gnss sensors in webots and urdf

File: asb_ros2_control/description/urdf/asb_description.urdf.xacro (robot description, xacro)
@@ -610,5 +610,5 @@
       <parent link="base_link"/>
       <child link="imu_link"/>
-      <origin xyz="0 0 0.23" rpy="0 0 0"/>
+      <origin xyz="0.133 -0.659 0.91" rpy="0 0 3.14159"/>
     </joint>
     <link name="inertial_link">
@@ -638,5 +638,5 @@
       <parent link="base_link"/>
       <child link="gnss_link"/>
-      <origin xyz="0.57 0 1.37" rpy="0 0 0"/>
+      <origin xyz="0.133 -0.659 0.91" rpy="0 0 3.14159"/>
     </joint>
     <!-- END generated by Webots -->

Commit message: added inertial unit in webots to implement GNSS compassing

File: asb_ros2_control/description/urdf/asb_description.urdf.xacro (robot description, xacro)
@@ -612,11 +612,4 @@
       <origin xyz="0.133 -0.659 0.91" rpy="0 0 3.14159"/>
     </joint>
-    <link name="inertial_link">
-    </link>
-    <joint name="imu_link_inertial_link_joint" type="fixed">
-      <parent link="imu_link"/>
-      <child link="inertial_link"/>
-      <origin xyz="0 0 0" rpy="0 0 0"/>
-    </joint>
     <link name="gyro_link">
     </link>
@@ -640,4 +633,11 @@
       <origin xyz="0.133 -0.659 0.91" rpy="0 0 3.14159"/>
     </joint>
+    <link name="inertial_link">
+    </link>
+    <joint name="base_link_inertial_link_joint" type="fixed">
+      <parent link="base_link"/>
+      <child link="inertial_link"/>
+      <origin xyz="0 0 0" rpy="0 0 0"/>
+    </joint>
     <!-- END generated by Webots -->
   </xacro:macro>

Commit message: dual antenna navsat_transform EKF setup

File: asb_ros2_control/description/urdf/asb_description.urdf.xacro (robot description, xacro)
@@ -631,5 +631,5 @@
       <parent link="base_link"/>
       <child link="gnss_link"/>
-      <origin xyz="0.133 -0.659 0.91" rpy="0 0 3.14159"/>
+      <origin xyz="0.133 -0.659 0.91" rpy="0 0 0"/>
     </joint>
     <link name="inertial_link">
