Commit message: implemented dual GNSS antenna in webots, repositioned vineyard

File: asb_ros2_control/description/urdf/asb_description.urdf.xacro (robot description, xacro)
@@ -370,4 +370,40 @@
         </geometry>
       </collision>
+      <visual>
+        <origin xyz="0.48 0 0.92" rpy="0 0 0"/>
+        <geometry>
+          <box size="0.31 0.8 0.8"/>
+        </geometry>
+      </visual>
+      <collision>
+        <origin xyz="0.48 0 0.92" rpy="0 0 0"/>
+        <geometry>
+          <box size="0.31 0.8 0.8"/>
+        </geometry>
+      </collision>
+      <visual>
+        <origin xyz="0.443 0.761 1.55188" rpy="0 0 0"/>
+        <geometry>
+          <box size="0.06 0.06 0.0225"/>
+        </geometry>
+      </visual>
+      <collision>
+        <origin xyz="0.443 0.761 1.55188" rpy="0 0 0"/>
+        <geometry>
+          <box size="0.06 0.06 0.0225"/>
+        </geometry>
+      </collision>
+      <visual>
+        <origin xyz="0.443 -0.656 1.55188" rpy="0 0 0"/>
+        <geometry>
+          <box size="0.06 0.06 0.0225"/>
+        </geometry>
+      </visual>
+      <collision>
+        <origin xyz="0.443 -0.656 1.55188" rpy="0 0 0"/>
+        <geometry>
+          <box size="0.06 0.06 0.0225"/>
+        </geometry>
+      </collision>
     </link>
     <link name="right_track">
@@ -626,10 +662,17 @@
       <origin xyz="0 0 0" rpy="0 0 0"/>
     </joint>
-    <link name="gnss_link">
-    </link>
-    <joint name="base_link_gnss_link_joint" type="fixed">
-      <parent link="base_link"/>
-      <child link="gnss_link"/>
-      <origin xyz="0.133 -0.659 0.91" rpy="0 0 0"/>
+    <link name="gnss_2_link">
+    </link>
+    <joint name="base_link_gnss_2_link_joint" type="fixed">
+      <parent link="base_link"/>
+      <child link="gnss_2_link"/>
+      <origin xyz="0.443 -0.656 1.54063" rpy="0 0 3.14159"/>
+    </joint>
+    <link name="gnss_1_link">
+    </link>
+    <joint name="base_link_gnss_1_link_joint" type="fixed">
+      <parent link="base_link"/>
+      <child link="gnss_1_link"/>
+      <origin xyz="0.443 0.761 1.54063" rpy="0 0 3.14159"/>
     </joint>
     <link name="inertial_link">

Commit message: fixed NTRIP client, GQ7 antenna offset and rob loc EKF params

File: asb_ros2_control/description/urdf/asb_description.urdf.xacro (robot description, xacro)
@@ -646,5 +646,5 @@
       <parent link="base_link"/>
       <child link="imu_link"/>
-      <origin xyz="0.133 -0.659 0.91" rpy="0 0 3.14159"/>
+      <origin xyz="0.133 -0.659 0.91" rpy="0 0 0"/>
     </joint>
     <link name="gyro_link">

Commit message: maybe improved gq7 measures

File: asb_ros2_control/description/urdf/asb_description.urdf.xacro (robot description, xacro)
@@ -383,5 +383,5 @@
       </collision>
       <visual>
-        <origin xyz="0.443 0.761 1.55188" rpy="0 0 0"/>
+        <origin xyz="0.443 -0.65586 1.55188" rpy="0 0 0"/>
         <geometry>
           <box size="0.06 0.06 0.0225"/>
@@ -389,5 +389,5 @@
       </visual>
       <collision>
-        <origin xyz="0.443 0.761 1.55188" rpy="0 0 0"/>
+        <origin xyz="0.443 -0.65586 1.55188" rpy="0 0 0"/>
         <geometry>
           <box size="0.06 0.06 0.0225"/>
@@ -395,5 +395,5 @@
       </collision>
       <visual>
-        <origin xyz="0.443 -0.656 1.55188" rpy="0 0 0"/>
+        <origin xyz="0.443 0.76114 1.55188" rpy="0 0 0"/>
         <geometry>
           <box size="0.06 0.06 0.0225"/>
@@ -401,5 +401,5 @@
       </visual>
       <collision>
-        <origin xyz="0.443 -0.656 1.55188" rpy="0 0 0"/>
+        <origin xyz="0.443 0.76114 1.55188" rpy="0 0 0"/>
         <geometry>
           <box size="0.06 0.06 0.0225"/>
@@ -646,5 +646,5 @@
       <parent link="base_link"/>
       <child link="imu_link"/>
-      <origin xyz="0.133 -0.659 0.91" rpy="0 0 0"/>
+      <origin xyz="0.03385 -0.69 0.91" rpy="0 0 0"/>
     </joint>
     <link name="gyro_link">
@@ -667,5 +667,5 @@
       <parent link="base_link"/>
       <child link="gnss_2_link"/>
-      <origin xyz="0.443 -0.656 1.54063" rpy="0 0 3.14159"/>
+      <origin xyz="0.443 0.76114 1.54063" rpy="0 0 0"/>
     </joint>
     <link name="gnss_1_link">
@@ -674,5 +674,5 @@
       <parent link="base_link"/>
       <child link="gnss_1_link"/>
-      <origin xyz="0.443 0.761 1.54063" rpy="0 0 3.14159"/>
+      <origin xyz="0.443 -0.65586 1.54063" rpy="0 0 0"/>
     </joint>
     <link name="inertial_link">

Commit message: fixed antenna and GQ7 measurement errors

File: asb_ros2_control/description/urdf/asb_description.urdf.xacro (robot description, xacro)
@@ -383,5 +383,5 @@
       </collision>
       <visual>
-        <origin xyz="0.443 -0.65586 1.55188" rpy="0 0 0"/>
+        <origin xyz="0.44185 -0.663 1.54363" rpy="0 0 0"/>
         <geometry>
           <box size="0.06 0.06 0.0225"/>
@@ -389,5 +389,5 @@
       </visual>
       <collision>
-        <origin xyz="0.443 -0.65586 1.55188" rpy="0 0 0"/>
+        <origin xyz="0.44185 -0.663 1.54363" rpy="0 0 0"/>
         <geometry>
           <box size="0.06 0.06 0.0225"/>
@@ -395,5 +395,5 @@
       </collision>
       <visual>
-        <origin xyz="0.443 0.76114 1.55188" rpy="0 0 0"/>
+        <origin xyz="0.44185 0.662 1.54363" rpy="0 0 0"/>
         <geometry>
           <box size="0.06 0.06 0.0225"/>
@@ -401,5 +401,5 @@
       </visual>
       <collision>
-        <origin xyz="0.443 0.76114 1.55188" rpy="0 0 0"/>
+        <origin xyz="0.44185 0.662 1.54363" rpy="0 0 0"/>
         <geometry>
           <box size="0.06 0.06 0.0225"/>
@@ -667,5 +667,5 @@
       <parent link="base_link"/>
       <child link="gnss_2_link"/>
-      <origin xyz="0.443 0.76114 1.54063" rpy="0 0 0"/>
+      <origin xyz="0.44185 0.662 1.54363" rpy="0 0 0"/>
     </joint>
     <link name="gnss_1_link">
@@ -674,5 +674,5 @@
       <parent link="base_link"/>
       <child link="gnss_1_link"/>
-      <origin xyz="0.443 -0.65586 1.54063" rpy="0 0 0"/>
+      <origin xyz="0.44185 -0.663 1.54363" rpy="0 0 0"/>
     </joint>
     <link name="inertial_link">

Commit message: set up front right OS0 lidar

File: asb_ros2_control/description/urdf/asb_description.urdf.xacro (robot description, xacro)
@@ -582,5 +582,5 @@
       <parent link="base_link"/>
       <child link="base_scan_rear_left_multilayer"/>
-      <origin xyz="-1 0.81 0.3" rpy="0 0 2.356194"/>
+      <origin xyz="-1 0.81 0.1859" rpy="0 0 -3.141593"/>
     </joint>
     <link name="base_scan_front_right_multilayer">
@@ -601,5 +601,5 @@
       <parent link="base_link"/>
       <child link="base_scan_front_right_multilayer"/>
-      <origin xyz="1 -0.81 0.3" rpy="0 0 -0.785398"/>
+      <origin xyz="0.9745 -0.81 0.1859" rpy="0 0 0"/>
     </joint>
     <link name="base_scan_rear_left">

Commit message: fixed sim LIDARs and remapped pointcloud topics

File: asb_ros2_control/description/urdf/asb_description.urdf.xacro (robot description, xacro)
@@ -565,17 +565,24 @@
       <origin xyz="0 0.44 0" rpy="0 0 0"/>
     </joint>
+    <link name="base_scan_rear_left_multilayer_sim">
+      <visual>
+        <origin xyz="0 0 0" rpy="0 0 0"/>
+        <geometry>
+          <cylinder radius="0.0435" length="0.0742"/>
+        </geometry>
+      </visual>
+      <collision>
+        <origin xyz="0 0 0" rpy="0 0 0"/>
+        <geometry>
+          <cylinder radius="0.0435" length="0.0742"/>
+        </geometry>
+      </collision>
+    </link>
+    <joint name="base_link_base_scan_rear_left_multilayer_sim_joint" type="fixed">
+      <parent link="base_link"/>
+      <child link="base_scan_rear_left_multilayer_sim"/>
+      <origin xyz="-1 0.81 0.1859" rpy="0 0 2.356194"/>
+    </joint>
     <link name="base_scan_rear_left_multilayer">
-      <visual>
-        <origin xyz="0 0 0" rpy="0 0 0"/>
-        <geometry>
-          <cylinder radius="0.0435" length="0.0742"/>
-        </geometry>
-      </visual>
-      <collision>
-        <origin xyz="0 0 0" rpy="0 0 0"/>
-        <geometry>
-          <cylinder radius="0.0435" length="0.0742"/>
-        </geometry>
-      </collision>
     </link>
     <joint name="base_link_base_scan_rear_left_multilayer_joint" type="fixed">
@@ -584,17 +591,24 @@
       <origin xyz="-1 0.81 0.1859" rpy="0 0 -3.141593"/>
     </joint>
+    <link name="base_scan_front_right_multilayer_sim">
+      <visual>
+        <origin xyz="0 0 0" rpy="0 0 0"/>
+        <geometry>
+          <cylinder radius="0.0435" length="0.0742"/>
+        </geometry>
+      </visual>
+      <collision>
+        <origin xyz="0 0 0" rpy="0 0 0"/>
+        <geometry>
+          <cylinder radius="0.0435" length="0.0742"/>
+        </geometry>
+      </collision>
+    </link>
+    <joint name="base_link_base_scan_front_right_multilayer_sim_joint" type="fixed">
+      <parent link="base_link"/>
+      <child link="base_scan_front_right_multilayer_sim"/>
+      <origin xyz="0.9745 -0.81 0.1859" rpy="0 0 -0.785398"/>
+    </joint>
     <link name="base_scan_front_right_multilayer">
-      <visual>
-        <origin xyz="0 0 0" rpy="0 0 0"/>
-        <geometry>
-          <cylinder radius="0.0435" length="0.0742"/>
-        </geometry>
-      </visual>
-      <collision>
-        <origin xyz="0 0 0" rpy="0 0 0"/>
-        <geometry>
-          <cylinder radius="0.0435" length="0.0742"/>
-        </geometry>
-      </collision>
     </link>
     <joint name="base_link_base_scan_front_right_multilayer_joint" type="fixed">

Commit message: placed OS0 lidar in front

File: asb_ros2_control/description/urdf/asb_description.urdf.xacro (robot description, xacro)
@@ -591,5 +591,5 @@
       <origin xyz="-1 0.81 0.1859" rpy="0 0 -3.141593"/>
     </joint>
-    <link name="base_scan_front_right_multilayer_sim">
+    <link name="base_scan_front_multilayer_sim">
       <visual>
         <origin xyz="0 0 0" rpy="0 0 0"/>
@@ -605,15 +605,15 @@
       </collision>
     </link>
-    <joint name="base_link_base_scan_front_right_multilayer_sim_joint" type="fixed">
-      <parent link="base_link"/>
-      <child link="base_scan_front_right_multilayer_sim"/>
-      <origin xyz="0.9745 -0.81 0.1859" rpy="0 0 -0.785398"/>
-    </joint>
-    <link name="base_scan_front_right_multilayer">
-    </link>
-    <joint name="base_link_base_scan_front_right_multilayer_joint" type="fixed">
-      <parent link="base_link"/>
-      <child link="base_scan_front_right_multilayer"/>
-      <origin xyz="0.9745 -0.81 0.1859" rpy="0 0 0"/>
+    <joint name="base_link_base_scan_front_multilayer_sim_joint" type="fixed">
+      <parent link="base_link"/>
+      <child link="base_scan_front_multilayer_sim"/>
+      <origin xyz="0.805 0 1.5359" rpy="-3.141593 0 0"/>
+    </joint>
+    <link name="base_scan_front_multilayer">
+    </link>
+    <joint name="base_link_base_scan_front_multilayer_joint" type="fixed">
+      <parent link="base_link"/>
+      <child link="base_scan_front_multilayer"/>
+      <origin xyz="0.805 0 1.5359" rpy="-3.141593 0 0"/>
     </joint>
     <link name="base_scan_rear_left">

Commit message: using multilayer lidar for obstacle avoidance and improved costmap footprints

File: asb_ros2_control/description/urdf/asb_description.urdf.xacro (robot description, xacro)
@@ -617,42 +617,4 @@
       <origin xyz="0.805 0 1.5359" rpy="-3.141593 0 0"/>
     </joint>
-    <link name="base_scan_rear_left">
-      <visual>
-        <origin xyz="0 0 -0.011" rpy="1.570741 0.000118 -1.570741"/>
-        <geometry>
-          <box size="0.06 0.087 0.06"/>
-        </geometry>
-      </visual>
-      <collision>
-        <origin xyz="0 0 -0.011" rpy="1.570741 0.000118 -1.570741"/>
-        <geometry>
-          <box size="0.06 0.087 0.06"/>
-        </geometry>
-      </collision>
-    </link>
-    <joint name="base_link_base_scan_rear_left_joint" type="fixed">
-      <parent link="base_link"/>
-      <child link="base_scan_rear_left"/>
-      <origin xyz="-1 0.81 0.4" rpy="0 0 2.356194"/>
-    </joint>
-    <link name="base_scan_front_right">
-      <visual>
-        <origin xyz="0 0 -0.011" rpy="1.570741 0.000118 -1.570741"/>
-        <geometry>
-          <box size="0.06 0.087 0.06"/>
-        </geometry>
-      </visual>
-      <collision>
-        <origin xyz="0 0 -0.011" rpy="1.570741 0.000118 -1.570741"/>
-        <geometry>
-          <box size="0.06 0.087 0.06"/>
-        </geometry>
-      </collision>
-    </link>
-    <joint name="base_link_base_scan_front_right_joint" type="fixed">
-      <parent link="base_link"/>
-      <child link="base_scan_front_right"/>
-      <origin xyz="1 -0.81 0.4" rpy="0 0 -0.785398"/>
-    </joint>
     <link name="imu_link">
     </link>

Commit message: added sprayer in webots robot model and URDF

File: asb_ros2_control/description/urdf/asb_description.urdf.xacro (robot description, xacro)
@@ -359,4 +359,16 @@
       </collision>
       <visual>
+        <origin xyz="0.48 0 0.92" rpy="0 0 0"/>
+        <geometry>
+          <box size="0.31 0.8 0.8"/>
+        </geometry>
+      </visual>
+      <collision>
+        <origin xyz="0.48 0 0.92" rpy="0 0 0"/>
+        <geometry>
+          <box size="0.31 0.8 0.8"/>
+        </geometry>
+      </collision>
+      <visual>
         <origin xyz="-0.15 0 0.88" rpy="0 0 0"/>
         <geometry>
@@ -371,13 +383,61 @@
       </collision>
       <visual>
-        <origin xyz="0.48 0 0.92" rpy="0 0 0"/>
-        <geometry>
-          <box size="0.31 0.8 0.8"/>
-        </geometry>
-      </visual>
-      <collision>
-        <origin xyz="0.48 0 0.92" rpy="0 0 0"/>
-        <geometry>
-          <box size="0.31 0.8 0.8"/>
+        <origin xyz="-0.8 0 0.87" rpy="3.141593 1.570793 3.141593"/>
+        <geometry>
+          <cylinder radius="0.3" length="0.53"/>
+        </geometry>
+      </visual>
+      <collision>
+        <origin xyz="-0.8 0 0.87" rpy="3.141593 1.570793 3.141593"/>
+        <geometry>
+          <cylinder radius="0.3" length="0.53"/>
+        </geometry>
+      </collision>
+      <visual>
+        <origin xyz="-1.11 0 0.595" rpy="0 0 0"/>
+        <geometry>
+          <box size="0.1 0.8 0.15"/>
+        </geometry>
+      </visual>
+      <collision>
+        <origin xyz="-1.11 0 0.595" rpy="0 0 0"/>
+        <geometry>
+          <box size="0.1 0.8 0.15"/>
+        </geometry>
+      </collision>
+      <visual>
+        <origin xyz="-1.11 0 1.145" rpy="0 0 0"/>
+        <geometry>
+          <box size="0.1 0.46 0.95"/>
+        </geometry>
+      </visual>
+      <collision>
+        <origin xyz="-1.11 0 1.145" rpy="0 0 0"/>
+        <geometry>
+          <box size="0.1 0.46 0.95"/>
+        </geometry>
+      </collision>
+      <visual>
+        <origin xyz="-1.11 0.077801 1.10525" rpy="0.17 0 0"/>
+        <geometry>
+          <box size="0.1 0.49 0.97"/>
+        </geometry>
+      </visual>
+      <collision>
+        <origin xyz="-1.11 0.077801 1.10525" rpy="0.17 0 0"/>
+        <geometry>
+          <box size="0.1 0.49 0.97"/>
+        </geometry>
+      </collision>
+      <visual>
+        <origin xyz="-1.11 -0.077801 1.10525" rpy="-0.17 0 0"/>
+        <geometry>
+          <box size="0.1 0.49 0.97"/>
+        </geometry>
+      </visual>
+      <collision>
+        <origin xyz="-1.11 -0.077801 1.10525" rpy="-0.17 0 0"/>
+        <geometry>
+          <box size="0.1 0.49 0.97"/>
         </geometry>
       </collision>
@@ -564,4 +624,11 @@
       <child link="left_track"/>
       <origin xyz="0 0.44 0" rpy="0 0 0"/>
+    </joint>
+    <link name="sprayer_link">
+    </link>
+    <joint name="base_link_sprayer_link_joint" type="fixed">
+      <parent link="base_link"/>
+      <child link="sprayer_link"/>
+      <origin xyz="-1.06 0 0.52" rpy="0 0 0"/>
     </joint>
     <link name="base_scan_rear_left_multilayer_sim">

Commit message: fixed high lidar message loss, added rear lidar in launch and config, fixed rear lidar names

File: asb_ros2_control/description/urdf/asb_description.urdf.xacro (robot description, xacro)
@@ -632,5 +632,5 @@
       <origin xyz="-1.06 0 0.52" rpy="0 0 0"/>
     </joint>
-    <link name="base_scan_rear_left_multilayer_sim">
+    <link name="base_scan_rear_multilayer_sim">
       <visual>
         <origin xyz="0 0 0" rpy="0 0 0"/>
@@ -646,14 +646,14 @@
       </collision>
     </link>
-    <joint name="base_link_base_scan_rear_left_multilayer_sim_joint" type="fixed">
-      <parent link="base_link"/>
-      <child link="base_scan_rear_left_multilayer_sim"/>
+    <joint name="base_link_base_scan_rear_multilayer_sim_joint" type="fixed">
+      <parent link="base_link"/>
+      <child link="base_scan_rear_multilayer_sim"/>
       <origin xyz="-1 0.81 0.1859" rpy="0 0 2.356194"/>
     </joint>
-    <link name="base_scan_rear_left_multilayer">
-    </link>
-    <joint name="base_link_base_scan_rear_left_multilayer_joint" type="fixed">
-      <parent link="base_link"/>
-      <child link="base_scan_rear_left_multilayer"/>
+    <link name="base_scan_rear_multilayer">
+    </link>
+    <joint name="base_link_base_scan_rear_multilayer_joint" type="fixed">
+      <parent link="base_link"/>
+      <child link="base_scan_rear_multilayer"/>
       <origin xyz="-1 0.81 0.1859" rpy="0 0 -3.141593"/>
     </joint>

Commit message: simplified lidar filter, fixed rear lidar position

File: asb_ros2_control/description/urdf/asb_description.urdf.xacro (robot description, xacro)
@@ -649,5 +649,5 @@
       <parent link="base_link"/>
       <child link="base_scan_rear_multilayer_sim"/>
-      <origin xyz="-1 0.81 0.1859" rpy="0 0 2.356194"/>
+      <origin xyz="-1 0 0.1859" rpy="0 0 -3.141593"/>
     </joint>
     <link name="base_scan_rear_multilayer">
@@ -656,5 +656,5 @@
       <parent link="base_link"/>
       <child link="base_scan_rear_multilayer"/>
-      <origin xyz="-1 0.81 0.1859" rpy="0 0 -3.141593"/>
+      <origin xyz="-1 0 0.1859" rpy="0 0 -3.141593"/>
     </joint>
     <link name="base_scan_front_multilayer_sim">
