Commit message: fixed front and rear lidar positions and improved sim model

File: asb_ros2_control/description/urdf/asb_description.urdf.xacro (robot description, xacro)
@@ -11,4 +11,172 @@
     <link name="base_link">
       <visual>
+        <origin xyz="0 0.77 1.515" rpy="0 0 0"/>
+        <geometry>
+          <box size="0.94 0.04 0.04"/>
+        </geometry>
+      </visual>
+      <collision>
+        <origin xyz="0 0.77 1.515" rpy="0 0 0"/>
+        <geometry>
+          <box size="0.94 0.04 0.04"/>
+        </geometry>
+      </collision>
+      <visual>
+        <origin xyz="0 -0.77 1.515" rpy="0 0 0"/>
+        <geometry>
+          <box size="0.94 0.04 0.04"/>
+        </geometry>
+      </visual>
+      <collision>
+        <origin xyz="0 -0.77 1.515" rpy="0 0 0"/>
+        <geometry>
+          <box size="0.94 0.04 0.04"/>
+        </geometry>
+      </collision>
+      <visual>
+        <origin xyz="0.49 0 1.515" rpy="0 0 0"/>
+        <geometry>
+          <box size="0.04 1.5 0.04"/>
+        </geometry>
+      </visual>
+      <collision>
+        <origin xyz="0.49 0 1.515" rpy="0 0 0"/>
+        <geometry>
+          <box size="0.04 1.5 0.04"/>
+        </geometry>
+      </collision>
+      <visual>
+        <origin xyz="-0.49 0 1.515" rpy="0 0 0"/>
+        <geometry>
+          <box size="0.04 1.5 0.04"/>
+        </geometry>
+      </visual>
+      <collision>
+        <origin xyz="-0.49 0 1.515" rpy="0 0 0"/>
+        <geometry>
+          <box size="0.04 1.5 0.04"/>
+        </geometry>
+      </collision>
+      <visual>
+        <origin xyz="0.175 0.06 1.555" rpy="0 0 0"/>
+        <geometry>
+          <box size="1.37 0.04 0.04"/>
+        </geometry>
+      </visual>
+      <collision>
+        <origin xyz="0.175 0.06 1.555" rpy="0 0 0"/>
+        <geometry>
+          <box size="1.37 0.04 0.04"/>
+        </geometry>
+      </collision>
+      <visual>
+        <origin xyz="0.175 -0.06 1.555" rpy="0 0 0"/>
+        <geometry>
+          <box size="1.37 0.04 0.04"/>
+        </geometry>
+      </visual>
+      <collision>
+        <origin xyz="0.175 -0.06 1.555" rpy="0 0 0"/>
+        <geometry>
+          <box size="1.37 0.04 0.04"/>
+        </geometry>
+      </collision>
+      <visual>
+        <origin xyz="-0.45 0.1325 0.236" rpy="0 0 0"/>
+        <geometry>
+          <box size="1.37 0.04 0.04"/>
+        </geometry>
+      </visual>
+      <collision>
+        <origin xyz="-0.45 0.1325 0.236" rpy="0 0 0"/>
+        <geometry>
+          <box size="1.37 0.04 0.04"/>
+        </geometry>
+      </collision>
+      <visual>
+        <origin xyz="-0.45 -0.1325 0.236" rpy="0 0 0"/>
+        <geometry>
+          <box size="1.37 0.04 0.04"/>
+        </geometry>
+      </visual>
+      <collision>
+        <origin xyz="-0.45 -0.1325 0.236" rpy="0 0 0"/>
+        <geometry>
+          <box size="1.37 0.04 0.04"/>
+        </geometry>
+      </collision>
+      <visual>
+        <origin xyz="-1.115 0 0.236" rpy="0 0 0"/>
+        <geometry>
+          <box size="0.04 0.225 0.04"/>
+        </geometry>
+      </visual>
+      <collision>
+        <origin xyz="-1.115 0 0.236" rpy="0 0 0"/>
+        <geometry>
+          <box size="0.04 0.225 0.04"/>
+        </geometry>
+      </collision>
+      <visual>
+        <origin xyz="-1.035 0 0.236" rpy="0 0 0"/>
+        <geometry>
+          <box size="0.04 0.225 0.04"/>
+        </geometry>
+      </visual>
+      <collision>
+        <origin xyz="-1.035 0 0.236" rpy="0 0 0"/>
+        <geometry>
+          <box size="0.04 0.225 0.04"/>
+        </geometry>
+      </collision>
+      <visual>
+        <origin xyz="0.49 0.77 0.86" rpy="0 0 0"/>
+        <geometry>
+          <box size="0.04 0.04 1.35"/>
+        </geometry>
+      </visual>
+      <collision>
+        <origin xyz="0.49 0.77 0.86" rpy="0 0 0"/>
+        <geometry>
+          <box size="0.04 0.04 1.35"/>
+        </geometry>
+      </collision>
+      <visual>
+        <origin xyz="0.49 -0.77 0.86" rpy="0 0 0"/>
+        <geometry>
+          <box size="0.04 0.04 1.35"/>
+        </geometry>
+      </visual>
+      <collision>
+        <origin xyz="0.49 -0.77 0.86" rpy="0 0 0"/>
+        <geometry>
+          <box size="0.04 0.04 1.35"/>
+        </geometry>
+      </collision>
+      <visual>
+        <origin xyz="-0.49 0.77 0.86" rpy="0 0 0"/>
+        <geometry>
+          <box size="0.04 0.04 1.35"/>
+        </geometry>
+      </visual>
+      <collision>
+        <origin xyz="-0.49 0.77 0.86" rpy="0 0 0"/>
+        <geometry>
+          <box size="0.04 0.04 1.35"/>
+        </geometry>
+      </collision>
+      <visual>
+        <origin xyz="-0.49 -0.77 0.86" rpy="0 0 0"/>
+        <geometry>
+          <box size="0.04 0.04 1.35"/>
+        </geometry>
+      </visual>
+      <collision>
+        <origin xyz="-0.49 -0.77 0.86" rpy="0 0 0"/>
+        <geometry>
+          <box size="0.04 0.04 1.35"/>
+        </geometry>
+      </collision>
+      <visual>
         <origin xyz="0.491 0 0.315" rpy="0 0 0"/>
         <geometry>
@@ -634,5 +802,5 @@
     <link name="base_scan_rear_multilayer_sim">
       <visual>
-        <origin xyz="0 0 0" rpy="0 0 0"/>
+        <origin xyz="0 0 0.04" rpy="0 0 0"/>
         <geometry>
           <cylinder radius="0.0435" length="0.0742"/>
@@ -640,5 +808,5 @@
       </visual>
       <collision>
-        <origin xyz="0 0 0" rpy="0 0 0"/>
+        <origin xyz="0 0 0.04" rpy="0 0 0"/>
         <geometry>
           <cylinder radius="0.0435" length="0.0742"/>
@@ -649,5 +817,5 @@
       <parent link="base_link"/>
       <child link="base_scan_rear_multilayer_sim"/>
-      <origin xyz="-1 0 0.1859" rpy="0 0 -3.141593"/>
+      <origin xyz="-1.075 0 0.2559" rpy="0 0 -3.141593"/>
     </joint>
     <link name="base_scan_rear_multilayer">
@@ -656,9 +824,9 @@
       <parent link="base_link"/>
       <child link="base_scan_rear_multilayer"/>
-      <origin xyz="-1 0 0.1859" rpy="0 0 -3.141593"/>
+      <origin xyz="-1.075 0 0.2559" rpy="0 0 -3.141593"/>
     </joint>
     <link name="base_scan_front_multilayer_sim">
       <visual>
-        <origin xyz="0 0 0" rpy="0 0 0"/>
+        <origin xyz="0 0 0.04" rpy="0 0 0"/>
         <geometry>
           <cylinder radius="0.0435" length="0.0742"/>
@@ -666,5 +834,5 @@
       </visual>
       <collision>
-        <origin xyz="0 0 0" rpy="0 0 0"/>
+        <origin xyz="0 0 0.04" rpy="0 0 0"/>
         <geometry>
           <cylinder radius="0.0435" length="0.0742"/>
@@ -675,5 +843,5 @@
       <parent link="base_link"/>
       <child link="base_scan_front_multilayer_sim"/>
-      <origin xyz="0.805 0 1.5359" rpy="-3.141593 0 0"/>
+      <origin xyz="0.8275 0 1.617" rpy="0 0.523599 0"/>
     </joint>
     <link name="base_scan_front_multilayer">
@@ -682,5 +850,5 @@
       <parent link="base_link"/>
       <child link="base_scan_front_multilayer"/>
-      <origin xyz="0.805 0 1.5359" rpy="-3.141593 0 0"/>
+      <origin xyz="0.8275 0 1.617" rpy="0 0.523599 0"/>
     </joint>
     <link name="imu_link">

Commit message: fixed lidar position and orientation, plus some ouster settings, added imu viz publisher

File: asb_ros2_control/description/urdf/asb_description.urdf.xacro (robot description, xacro)
@@ -59,25 +59,25 @@
       </collision>
       <visual>
-        <origin xyz="0.175 0.06 1.555" rpy="0 0 0"/>
-        <geometry>
-          <box size="1.37 0.04 0.04"/>
-        </geometry>
-      </visual>
-      <collision>
-        <origin xyz="0.175 0.06 1.555" rpy="0 0 0"/>
-        <geometry>
-          <box size="1.37 0.04 0.04"/>
-        </geometry>
-      </collision>
-      <visual>
-        <origin xyz="0.175 -0.06 1.555" rpy="0 0 0"/>
-        <geometry>
-          <box size="1.37 0.04 0.04"/>
-        </geometry>
-      </visual>
-      <collision>
-        <origin xyz="0.175 -0.06 1.555" rpy="0 0 0"/>
-        <geometry>
-          <box size="1.37 0.04 0.04"/>
+        <origin xyz="0.165 0.04 1.555" rpy="0 0 0"/>
+        <geometry>
+          <box size="1.32 0.04 0.04"/>
+        </geometry>
+      </visual>
+      <collision>
+        <origin xyz="0.165 0.04 1.555" rpy="0 0 0"/>
+        <geometry>
+          <box size="1.32 0.04 0.04"/>
+        </geometry>
+      </collision>
+      <visual>
+        <origin xyz="0.165 -0.04 1.555" rpy="0 0 0"/>
+        <geometry>
+          <box size="1.32 0.04 0.04"/>
+        </geometry>
+      </visual>
+      <collision>
+        <origin xyz="0.165 -0.04 1.555" rpy="0 0 0"/>
+        <geometry>
+          <box size="1.32 0.04 0.04"/>
         </geometry>
       </collision>
@@ -802,5 +802,5 @@
     <link name="base_scan_rear_multilayer_sim">
       <visual>
-        <origin xyz="0 0 0.04" rpy="0 0 0"/>
+        <origin xyz="0 0 0" rpy="0 0 0"/>
         <geometry>
           <cylinder radius="0.0435" length="0.0742"/>
@@ -808,5 +808,5 @@
       </visual>
       <collision>
-        <origin xyz="0 0 0.04" rpy="0 0 0"/>
+        <origin xyz="0 0 0" rpy="0 0 0"/>
         <geometry>
           <cylinder radius="0.0435" length="0.0742"/>
@@ -817,16 +817,30 @@
       <parent link="base_link"/>
       <child link="base_scan_rear_multilayer_sim"/>
+      <origin xyz="-1.075 0 0.316595" rpy="0 0 -3.141593"/>
+    </joint>
+    <link name="base_scan_rear_multilayer_plate_optical_center">
+    </link>
+    <joint name="base_link_base_scan_rear_multilayer_plate_optical_center_joint" type="fixed">
+      <parent link="base_link"/>
+      <child link="base_scan_rear_multilayer_plate_optical_center"/>
+      <origin xyz="-1.075 0 0.316595" rpy="0 0 -3.141593"/>
+    </joint>
+    <link name="base_scan_rear_multilayer_plate_top">
+    </link>
+    <joint name="base_link_base_scan_rear_multilayer_plate_top_joint" type="fixed">
+      <parent link="base_link"/>
+      <child link="base_scan_rear_multilayer_plate_top"/>
+      <origin xyz="-1.075 0 0.2784" rpy="0 0 -3.141593"/>
+    </joint>
+    <link name="base_scan_rear_multilayer_plate_bottom">
+    </link>
+    <joint name="base_link_base_scan_rear_multilayer_plate_bottom_joint" type="fixed">
+      <parent link="base_link"/>
+      <child link="base_scan_rear_multilayer_plate_bottom"/>
       <origin xyz="-1.075 0 0.2559" rpy="0 0 -3.141593"/>
     </joint>
-    <link name="base_scan_rear_multilayer">
-    </link>
-    <joint name="base_link_base_scan_rear_multilayer_joint" type="fixed">
-      <parent link="base_link"/>
-      <child link="base_scan_rear_multilayer"/>
-      <origin xyz="-1.075 0 0.2559" rpy="0 0 -3.141593"/>
-    </joint>
     <link name="base_scan_front_multilayer_sim">
       <visual>
-        <origin xyz="0 0 0.04" rpy="0 0 0"/>
+        <origin xyz="0 0 0" rpy="0 0 0"/>
         <geometry>
           <cylinder radius="0.0435" length="0.0742"/>
@@ -834,5 +848,5 @@
       </visual>
       <collision>
-        <origin xyz="0 0 0.04" rpy="0 0 0"/>
+        <origin xyz="0 0 0" rpy="0 0 0"/>
         <geometry>
           <cylinder radius="0.0435" length="0.0742"/>
@@ -843,12 +857,26 @@
       <parent link="base_link"/>
       <child link="base_scan_front_multilayer_sim"/>
-      <origin xyz="0.8275 0 1.617" rpy="0 0.523599 0"/>
-    </joint>
-    <link name="base_scan_front_multilayer">
-    </link>
-    <joint name="base_link_base_scan_front_multilayer_joint" type="fixed">
-      <parent link="base_link"/>
-      <child link="base_scan_front_multilayer"/>
-      <origin xyz="0.8275 0 1.617" rpy="0 0.523599 0"/>
+      <origin xyz="0.856063 0.000607 1.67055" rpy="-0.01 0.49 0"/>
+    </joint>
+    <link name="base_scan_front_multilayer_optical_center">
+    </link>
+    <joint name="base_link_base_scan_front_multilayer_optical_center_joint" type="fixed">
+      <parent link="base_link"/>
+      <child link="base_scan_front_multilayer_optical_center"/>
+      <origin xyz="0.856063 0.000607 1.67055" rpy="-0.01 0.49 0"/>
+    </joint>
+    <link name="base_scan_front_multilayer_plate_top">
+    </link>
+    <joint name="base_link_base_scan_front_multilayer_plate_top_joint" type="fixed">
+      <parent link="base_link"/>
+      <child link="base_scan_front_multilayer_plate_top"/>
+      <origin xyz="0.838089 0.000225 1.636852" rpy="-0.01 0.49 0"/>
+    </joint>
+    <link name="base_scan_front_multilayer_plate_bottom">
+    </link>
+    <joint name="base_link_base_scan_front_multilayer_plate_bottom_joint" type="fixed">
+      <parent link="base_link"/>
+      <child link="base_scan_front_multilayer_plate_bottom"/>
+      <origin xyz="0.8275 0 1.617" rpy="-0.01 0.49 0"/>
     </joint>
     <link name="imu_link">

Commit message: added frame for ST VL53L8 depth sensor

File: asb_ros2_control/description/urdf/asb_description.urdf.xacro (robot description, xacro)
@@ -880,4 +880,11 @@
       <origin xyz="0.8275 0 1.617" rpy="-0.01 0.49 0"/>
     </joint>
+    <link name="VL53L8">
+    </link>
+    <joint name="base_link_VL53L8_joint" type="fixed">
+      <parent link="base_link"/>
+      <child link="VL53L8"/>
+      <origin xyz="0.49 -0.5 1.515" rpy="-1.570799 0.000001 -1.570795"/>
+    </joint>
     <link name="imu_link">
     </link>
